Commit message: Finished model

File: src/romi_soccer/models/romi/romi.urdf (robot description, URDF)
Before this commit: robot romi, 3 links, 2 joints
Links:
- link chassis: geometry collision cylinder length=0.007 radius=0.015; collision cylinder length=0.007 radius=0.015
Joints:
- joint wheel_l_joint: axis 0 0 1 -> 1 0 0; origin xyz=0 0 0 rpy=0 0 0 -> xyz=0.0815 0.077 0.091 rpy=0 0 0
- joint wheel_r_joint: axis 0 0 1 -> 1 0 0; origin xyz=0 0 0 rpy=0 0 0 -> xyz=-0.06 0.077 0.091 rpy=0 0 0

Commit message: Updates

File: src/romi_soccer/models/romi/romi.urdf (robot description, URDF)
Before this commit: robot romi, 3 links, 2 joints
Links:
- link chassis: mass 0.160 -> 0.146
Joints:
- joint wheel_l_joint: origin xyz=0.0815 0.077 0.091 rpy=0 0 0 -> xyz=0.0815 0.085 0.09 rpy=0 0 0
- joint wheel_r_joint: origin xyz=-0.06 0.077 0.091 rpy=0 0 0 -> xyz=-0.06 0.085 0.09 rpy=0 0 0

Commit message: json grabber updates

File: src/romi_soccer/models/romi/romi.urdf (robot description, URDF)
Before this commit: robot romi, 3 links, 2 joints
Links:
- added link dummy
Joints:
- added joint dummy_joint: type fixed, parent chassis, child dummy
